Commit message: AV v8: R55–R57 perf ratchets, CoG fix (base under the load), standard home view, docs
- R55 step fly-ins at interaction resolution, clock clamped 50 ms/frame (every step moves mid-animation)
- R56 CSS variables cached; R57 0.75x interaction rung + double step when far over budget
- servo mount: base 80x54 under the load, shaft +4 mm -> CoG 12.1 mm inside the footprint (was 8 mm outside)
- research_v8, ADR_v8, DESIGN_BRIEF, DESIGN_DECISIONS, SKILL_UPDATE_v8, MARKETING_v8

Co-Authored-By: Claude Opus 5.5 <noreply@anthropic.com>
Claude-Session: https://claude.ai/code/session_015TiuMNVcJGucZKHjohAHfr

File: sp_av_v6_bundle/examples/v8_demo/out/servo_mount_v1.urdf (robot description, URDF)
Before this commit: robot servo_mount_v1, 3 links, 2 joints
Links:
- link base_link: mass 0.037828 -> 0.045848
Joints:
- joint shaft: origin xyz=-0.005300 -0.014000 0.048000 rpy=0 0 0 -> xyz=-0.005300 -0.014000 0.052000 rpy=0 0 0
